Commit message: change continuous to revolute

File: urdf/robokit_mv.urdf (robot description, URDF)
Before this commit: robot Robokit-MV, 30 links, 29 joints
Joints:
- joint head_pitch: limit effort=2.5 velocity=8 -> lower=-0.65 upper=1.61 effort=2.5 velocity=8; type continuous -> revolute
- joint head_yaw: limit effort=2.5 velocity=8 -> lower=-2.3 upper=2.3 effort=2.5 velocity=8; type continuous -> revolute
- joint left_ankle_pitch: limit effort=2.5 velocity=8 -> lower=-1 upper=1.8 effort=2.5 velocity=8; type continuous -> revolute
- joint left_ankle_roll: limit effort=2.5 velocity=8 -> lower=-1.51 upper=0.3 effort=2.5 velocity=8; type continuous -> revolute
- joint left_elbow: limit effort=2.5 velocity=8 -> lower=-0.55 upper=2.0 effort=2.5 velocity=8; type continuous -> revolute
- joint left_hip_pitch: type continuous -> revolute
- joint left_hip_roll: limit effort=2.5 velocity=8 -> lower=-0.42 upper=2.5 effort=2.5 velocity=8; type continuous -> revolute
- joint left_hip_yaw: limit effort=2.5 velocity=8 -> lower=-1.64 upper=1.81 effort=2.5 velocity=8; type continuous -> revolute
- joint left_knee: limit effort=2.5 velocity=8 -> lower=-0.9 upper=2.1 effort=2.5 velocity=8; type continuous -> revolute
- joint left_shoulder_pitch: limit effort=2.5 velocity=8 -> lower=-1.51 upper=0.3 effort=2.5 velocity=8; type continuous -> revolute
- joint left_shoulder_roll: limit effort=2.5 velocity=8 -> lower=-3.0 upper=0.60 effort=2.5 velocity=8; type continuous -> revolute
- joint left_shoulder_twirl: limit effort=2.5 velocity=8 -> lower=-2 upper=2 effort=2.5 velocity=8; type continuous -> revolute
- joint pelvis_yaw: limit effort=2.5 velocity=8 -> lower=-1.53 upper=2.0 effort=2.5 velocity=8; type continuous -> revolute
- joint right_anke_roll: limit effort=2.5 velocity=8 -> lower=-1.51 upper=0.3 effort=2.5 velocity=8; type continuous -> revolute
- joint right_ankle_pitch: limit effort=2.5 velocity=8 -> lower=-1 upper=1.8 effort=2.5 velocity=8; type continuous -> revolute
- joint right_elbow: limit effort=2.5 velocity=8 -> lower=-0.55 upper=2.0 effort=2.5 velocity=8; type continuous -> revolute
- joint right_hip_pitch: limit lower=-2.0 upper=2.0 effort=2.5 velocity=8 -> lower=-1.8 upper=1.95 effort=2.5 velocity=8; type continuous -> revolute
- joint right_hip_roll: limit effort=2.5 velocity=8 -> lower=-0.42 upper=2.5 effort=2.5 velocity=8; type continuous -> revolute
- joint right_hip_yaw: limit effort=2.5 velocity=8 -> lower=-1.64 upper=1.81 effort=2.5 velocity=8; type continuous -> revolute
- joint right_knee: limit effort=2.5 velocity=8 -> lower=-0.9 upper=2.1 effort=2.5 velocity=8; type continuous -> revolute
- joint right_shoulder_pitch: limit effort=2.5 velocity=8 -> lower=-1.51 upper=1.51 effort=2.5 velocity=8; type continuous -> revolute
- joint right_shoulder_roll: limit effort=2.5 velocity=8 -> lower=-3.0 upper=0.60 effort=2.5 velocity=8; type continuous -> revolute
- joint right_shoulder_twirl: limit effort=2.5 velocity=8 -> lower=-2 upper=2 effort=2.5 velocity=8; type continuous -> revolute
